File: Guitarpedal.kicad_pcb (KiCad board)
At the start: 4 copper layers, 60 x 90 mm, 68 parts, among them J1 AudioJack2, J2 AudioJack2, SW1 SW_SPDT, SW2 SW_SPDT, U1 TL072, U2 TL072, U3 TL072, U4 3PDT_footswitch

Commit message: Updated to 6.0
Other:
- net class Default removed
